File: AD7766_dev_board.sch (KiCad schematic (older format))
At the start: 67 parts, among them J1 Conn_Coaxial, J2 Conn_Coaxial, J3 Conn_01x06_Male, J4 Conn_01x10_Male, U1 PWR_JACK_POS, U2 PWR_JACK_GND, U3 ADR445, U4 ADP3330-5, U5 ADP3330-2.5, U6 ADP3330-2.5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

Commit message: updated PCB to add voltage divider to SYNC/PD pin
Parts:
- added R? (x2): R_US, symbol Device:R_US
- C6: value 100nF -> 10uF
- R1: value 3k -> 30k
- R2, R4, R5: value 1k -> 10k
Connections:
- wire segments 174 -> 177
Changed lines of the file:
@@
 P 3300 4450
 F 0 "C6" H 3415 4496 50  0000 L CNN
-F 1 "100nF" H 3415 4405 50  0000 L CNN
+F 1 "10uF" H 3415 4405 50  0000 L CNN
 F 2 "Capacitor_SMD:C_0805_2012Metric_Pad1.15x1.40mm_HandSolder" H 3338 4300 50  0001 C CNN
 F 3 "~" H 3300 4450 50  0001 C CNN
@@
 P 3800 4400
 F 0 "R1" H 3868 4446 50  0000 L CNN
-F 1 "3k" H 3868 4355 50  0000 L CNN
+F 1 "30k" H 3868 4355 50  0000 L CNN
 F 2 "Resistor_SMD:R_0805_2012Metric_Pad1.15x1.40mm_HandSolder" V 3840 4390 50  0001 C CNN
 F 3 "~" H 3800 4400 50  0001 C CNN
@@
 P 3800 4750
 F 0 "R2" H 3868 4796 50  0000 L CNN
-F 1 "1k" H 3868 4705 50  0000 L CNN
+F 1 "10k" H 3868 4705 50  0000 L CNN
 F 2 "Resistor_SMD:R_0805_2012Metric_Pad1.15x1.40mm_HandSolder" V 3840 4740 50  0001 C CNN
 F 3 "~" H 3800 4750 50  0001 C CNN
@@
 P 4450 4400
 F 0 "R4" H 4518 4446 50  0000 L CNN
-F 1 "1k" H 4518 4355 50  0000 L CNN
+F 1 "10k" H 4518 4355 50  0000 L CNN
 F 2 "Resistor_SMD:R_0805_2012Metric_Pad1.15x1.40mm_HandSolder" V 4490 4390 50  0001 C CNN
 F 3 "~" H 4450 4400 50  0001 C CNN
@@
 P 4450 4750
 F 0 "R5" H 4518 4796 50  0000 L CNN
-F 1 "1k" H 4518 4705 50  0000 L CNN
+F 1 "10k" H 4518 4705 50  0000 L CNN
 F 2 "Resistor_SMD:R_0805_2012Metric_Pad1.15x1.40mm_HandSolder" V 4490 4740 50  0001 C CNN
 F 3 "~" H 4450 4750 50  0001 C CNN
@@
 NoConn ~ 6650 2150
 NoConn ~ 8850 1350
-Text Label 6350 1750 0    50   ~ 0
-SYNCPD
 NoConn ~ 8850 1450
 NoConn ~ 8850 1550
@@
 Wire Wire Line
 	5350 1250 6000 1250
-Wire Wire Line
-	5650 2050 6650 2050
 Wire Wire Line
 	5850 1950 6650 1950
@@
 	5500 1850 5050 1850
 Connection ~ 5500 1850
+Wire Wire Line
+	5950 1750 5650 1750
+$Comp
+L power:GND #PWR0103
+U 1 1 5FFF39E7
+P 5650 2500
+F 0 "#PWR0103" H 5650 2250 50  0001 C CNN
+F 1 "GND" H 5655 2327 50  0000 C CNN
+F 2 "" H 5650 2500 50  0001 C CNN
+F 3 "" H 5650 2500 50  0001 C CNN
+	1    5650 2500
+	1    0    0    -1
+$EndComp
+Wire Wire Line
+	5650 1750 5650 2200
+Wire Wire Line
+	6650 2050 6250 2050
+Wire Wire Line
+	5650 1750 5400 1750
+Connection ~ 5650 1750
+$Comp
+L Device:R_US R?
+U 1 1 5FFF3448
+P 5650 2350
+F 0 "R?" H 5718 2396 50  0000 L CNN
+F 1 "R_US" H 5718 2305 50  0000 L CNN
+F 2 "" V 5690 2340 50  0001 C CNN
+F 3 "~" H 5650 2350 50  0001 C CNN
+	1    5650 2350
+	1    0    0    -1
+$EndComp
+$Comp
+L Device:R_US R?
+U 1 1 5FFE825F
+P 6100 1750
+F 0 "R?" V 5895 1750 50  0000 C CNN
+F 1 "R_US" V 5986 1750 50  0000 C CNN
+F 2 "" V 6140 1740 50  0001 C CNN
+F 3 "~" H 6100 1750 50  0001 C CNN
+	1    6100 1750
+	0    1    1    0
+$EndComp
+Text Label 6350 1750 0    50   ~ 0
+SYNCPD
 $EndSCHEMATC

Commit message: updated AD7766 dev board schematic, README
Parts:
- U1: symbol my_library:PWR_JACK_POS -> AD7766_dev_board-rescue:PWR_JACK_POS-my_library
- U2: symbol my_library:PWR_JACK_GND -> AD7766_dev_board-rescue:PWR_JACK_GND-my_library
Changed lines of the file:
@@
 	6400 5350 6500 5350
 $Comp
-L my_library:PWR_JACK_POS U1
+L AD7766_dev_board-rescue:PWR_JACK_POS-my_library U1
 U 1 1 5F7320F5
 P 1450 5850
@@
 $EndComp
 $Comp
-L my_library:PWR_JACK_GND U2
+L AD7766_dev_board-rescue:PWR_JACK_GND-my_library U2
 U 1 1 5F73473B
 P 1450 6300
